File: Chapter 1/Zener/Zener.kicad_sch (KiCad schematic)
At the start: 3 parts

Commit message: added v out tags to Chapter 1
Connections:
- net Vout renamed V-out
Changed lines of the file:
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@@
-(kicad_sch (version 20210406) (generator eeschema)
+(kicad_sch (version 20211123) (generator eeschema)
   (paper "A4")
-  (junction (at 63.5 55.88) (diameter 1.016) (color 0 0 0 0))
-  (wire (pts (xy 50.8 35.56) (xy 58.42 35.56))
+  (junction (at 63.5 55.88) (diameter 1.016) (color 0 0 0 0)
+  )
+  (wire (pts (xy 63.5 55.88) (xy 73.66 55.88))
     (stroke (width 0) (type solid) (color 0 0 0 0))
   )
@@
     (stroke (width 0) (type solid) (color 0 0 0 0))
   )
-  (wire (pts (xy 50.8 53.34) (xy 50.8 55.88))
-    (stroke (width 0) (type solid) (color 0 0 0 0))
-  )
-  (wire (pts (xy 50.8 55.88) (xy 63.5 55.88))
-    (stroke (width 0) (type solid) (color 0 0 0 0))
-  )
-  (wire (pts (xy 63.5 55.88) (xy 73.66 55.88))
+  (wire (pts (xy 66.04 35.56) (xy 73.66 35.56))
     (stroke (width 0) (type solid) (color 0 0 0 0))
   )
   (wire (pts (xy 63.5 63.5) (xy 63.5 55.88))
-    (stroke (width 0) (type solid) (color 0 0 0 0))
-  )
-  (wire (pts (xy 66.04 35.56) (xy 73.66 35.56))
     (stroke (width 0) (type solid) (color 0 0 0 0))
   )
@@
     (stroke (width 0) (type solid) (color 0 0 0 0))
   )
+  (wire (pts (xy 50.8 55.88) (xy 63.5 55.88))
+    (stroke (width 0) (type solid) (color 0 0 0 0))
+  )
+  (wire (pts (xy 50.8 53.34) (xy 50.8 55.88))
+    (stroke (width 0) (type solid) (color 0 0 0 0))
+  )
+  (wire (pts (xy 50.8 35.56) (xy 58.42 35.56))
+    (stroke (width 0) (type solid) (color 0 0 0 0))
+  )
   (text ".model DIODE d(Bv=5.6)\n.dc V1 -50 50 1" (at 68.58 25.4 0)
     (effects (font (size 1.27 1.27)) (justify left bottom))
+  )
+  (label "Vout" (at 73.66 35.56 180)
+    (effects (font (size 1.27 1.27)) (justify right bottom))
   )
   (label "Vin" (at 52.07 35.56 180)
     (effects (font (size 1.27 1.27)) (justify right bottom))
   )
-  (label "Vout" (at 73.66 35.56 180)
-    (effects (font (size 1.27 1.27)) (justify right bottom))
+  (global_label "V-out" (shape input) (at 73.66 35.56 0) (fields_autoplaced)
+    (effects (font (size 1.27 1.27)) (justify left))
+    (property "Intersheet References" "${INTERSHEET_REFS}" (id 0) (at 81.9484 35.4806 0)
+      (effects (font (size 1.27 1.27)) (justify left) hide)
+    )
+  )
+  (symbol (lib_id "Zener-rescue:VSOURCE-pspice") (at 50.8 45.72 0) (unit 1)
+    (in_bom yes) (on_board yes)
+    (property "Reference" "V1" (id 0) (at 56.5912 44.5516 0)
+      (effects (font (size 1.27 1.27)) (justify left))
+    )
+    (property "Value" "dc 0" (id 1) (at 56.5912 46.863 0)
+      (effects (font (size 1.27 1.27)) (justify left))
+    )
+    (property "Footprint" "" (id 2) (at 50.8 45.72 0)
+      (effects (font (size 1.27 1.27)) hide)
+    )
+    (property "Datasheet" "~" (id 3) (at 50.8 45.72 0)
+      (effects (font (size 1.27 1.27)) hide)
+    )
+    (pin "1")
+    (pin "2")
+  )
+  (symbol (lib_id "Zener-rescue:R-Device") (at 62.23 35.56 270) (unit 1)
+    (in_bom yes) (on_board yes)
+    (property "Reference" "R1" (id 0) (at 62.23 30.3022 90))
+    (property "Value" "10k" (id 1) (at 62.23 32.6136 90))
+    (property "Footprint" "" (id 2) (at 62.23 33.782 90)
+      (effects (font (size 1.27 1.27)) hide)
+    )
+    (property "Datasheet" "~" (id 3) (at 62.23 35.56 0)
+      (effects (font (size 1.27 1.27)) hide)
+    )
+    (pin "1")
+    (pin "2")
   )
   (symbol (lib_id "Zener-rescue:0-pspice") (at 63.5 63.5 0) (unit 1)
@@
     (pin "1")
   )
-  (symbol (lib_id "Zener-rescue:R-Device") (at 62.23 35.56 270) (unit 1)
-    (in_bom yes) (on_board yes)
-    (property "Reference" "R1" (id 0) (at 62.23 30.3022 90))
-    (property "Value" "10k" (id 1) (at 62.23 32.6136 90))
-    (property "Footprint" "" (id 2) (at 62.23 33.782 90)
-      (effects (font (size 1.27 1.27)) hide)
-    )
-    (property "Datasheet" "~" (id 3) (at 62.23 35.56 0)
-      (effects (font (size 1.27 1.27)) hide)
-    )
-    (pin "1")
-    (pin "2")
-  )
   (symbol (lib_id "pspice:DIODE") (at 73.66 41.91 90) (unit 1)
     (in_bom yes) (on_board yes) (fields_autoplaced)
@@
       (effects (font (size 1.27 1.27)) hide)
     )
-    (pin "1")
-    (pin "2")
-  )
-  (symbol (lib_id "Zener-rescue:VSOURCE-pspice") (at 50.8 45.72 0) (unit 1)
-    (in_bom yes) (on_board yes)
-    (property "Reference" "V1" (id 0) (at 56.5912 44.5516 0)
-      (effects (font (size 1.27 1.27)) (justify left))
-    )
-    (property "Value" "dc 0" (id 1) (at 56.5912 46.863 0)
-      (effects (font (size 1.27 1.27)) (justify left))
-    )
-    (property "Footprint" "" (id 2) (at 50.8 45.72 0)
-      (effects (font (size 1.27 1.27)) hide)
-    )
-    (property "Datasheet" "~" (id 3) (at 50.8 45.72 0)
-      (effects (font (size 1.27 1.27)) hide)
-    )
